Commit message: found a workaround for gazebo bug

File: julie/julie_description/urdf/julie_chassis.urdf.xacro (robot description, xacro)
@@ -7,5 +7,5 @@
       <visual>
         <xacro:if value="${chassis_hq_visual}">
-	  <origin xyz="0.33 0 -0.6" rpy="0 0 0"/>
+	  <origin xyz="0.03 0 -0.3" rpy="0 0 0"/>
           <geometry>
             <mesh filename="package://julie_description/meshes/chassis.dae"/>
